File: hardware/freakduino-alt.sch (KiCad schematic (older format))
At the start: 10 parts, among them U6 ATMEGA328-QFP32

Commit message: Laboriously re-worked schematic and 3D settings for KiCAD v5+
Parts:
- C13, C20, C22, C23: symbol C -> Device:C
- R11, R13, R14, R15: symbol R -> Device:R
- S2: symbol PBS_SMD -> freakduino:PBS_SMD
- U6: symbol ATMEGA328-QFP32 -> freakduino:ATMEGA328-QFP32
Connections:
- wire segments 58 -> 71
Changed lines of the file:
@@
-EESchema Schematic File Version 2
-LIBS:freakduino
-LIBS:power
-LIBS:device
-LIBS:transistors
-LIBS:conn
-LIBS:linear
-LIBS:regul
-LIBS:74xx
-LIBS:cmos4000
-LIBS:adc-dac
-LIBS:memory
-LIBS:xilinx
-LIBS:special
-LIBS:microcontrollers
-LIBS:dsp
-LIBS:microchip
-LIBS:analog_switches
-LIBS:motorola
-LIBS:texas
-LIBS:intel
-LIBS:audio
-LIBS:interface
-LIBS:digital-audio
-LIBS:philips
-LIBS:display
-LIBS:cypress
-LIBS:siliconi
-LIBS:opto
-LIBS:atmel
-LIBS:contrib
-LIBS:valves
+EESchema Schematic File Version 4
 LIBS:freakduino-alt-cache
-EELAYER 27 0
+EELAYER 26 0
 EELAYER END
 $Descr A4 11693 8268
@@
 NoConn ~ 6900 3850
 $Comp
-L R R13
+L Device:R R13
 U 1 1 51E29D02
 P 5650 2350
@@
 $EndComp
 $Comp
-L PBS_SMD S2
+L freakduino:PBS_SMD S2
 U 1 1 51E2A061
 P 5150 2800
 F 0 "S2" H 5050 3200 60  0000 C CNN
-F 1 "PBS_SMD" H 5150 2550 60  0000 C CNN
+F 1 "PBS_SMD" H 5150 2550 60  0001 C CNN
 F 2 "" H 5150 2800 60  0000 C CNN
 F 3 "" H 5150 2800 60  0000 C CNN
@@
 $EndComp
 $Comp
-L VSS #PWR01
+L power:VSS #PWR01
 U 1 1 51E2A09E
-P 4600 3100
-F 0 "#PWR01" H 4600 3100 30  0001 C CNN
-F 1 "VSS" H 4600 3030 30  0000 C CNN
-F 2 "" H 4600 3100 60  0000 C CNN
-F 3 "" H 4600 3100 60  0000 C CNN
-	1    4600 3100
-	1    0    0    -1
+P 4600 3000
+F 0 "#PWR01" H 4600 3000 30  0001 C CNN
+F 1 "VSS" H 4600 3150 30  0000 C CNN
+F 2 "" H 4600 3000 60  0000 C CNN
+F 3 "" H 4600 3000 60  0000 C CNN
+	1    4600 3000
+	-1   0    0    1
 $EndComp
 Text Label 6250 3150 0    60   ~ 0
 RESET_N
 $Comp
-L C C13
+L Device:C C13
 U 1 1 51E2A127
 P 6000 2350
@@
 DTR_N
 $Comp
-L R R14
+L Device:R R14
 U 1 1 51E2A219
 P 5950 5400
@@
 $EndComp
 $Comp
-L R R15
+L Device:R R15
 U 1 1 51E2A226
 P 5950 5500
@@
 VBAT
 $Comp
-L VSS #PWR02
+L power:VSS #PWR02
 U 1 1 51E2A474
-P 7700 6250
-F 0 "#PWR02" H 7700 6250 30  0001 C CNN
-F 1 "VSS" H 7700 6180 30  0000 C CNN
-F 2 "" H 7700 6250 60  0000 C CNN
-F 3 "" H 7700 6250 60  0000 C CNN
-	1    7700 6250
-	1    0    0    -1
-$EndComp
-Wire Wire Line
-	5650 2600 5650 2900
+P 7700 6150
+F 0 "#PWR02" H 7700 6150 30  0001 C CNN
+F 1 "VSS" H 7700 6300 30  0000 C CNN
+F 2 "" H 7700 6150 60  0000 C CNN
+F 3 "" H 7700 6150 60  0000 C CNN
+	1    7700 6150
+	-1   0    0    1
+$EndComp
+Wire Wire Line
+	5650 2500 5650 2700
 Connection ~ 5650 2700
 Wire Wire Line
@@
 	4750 2700 4600 2700
 Wire Wire Line
-	4600 2700 4600 3100
+	4600 2700 4600 2900
 Wire Wire Line
 	4750 2900 4600 2900
 Connection ~ 4600 2900
 Wire Wire Line
-	5650 2100 5650 2000
-Wire Wire Line
-	6000 2550 6000 3450
+	5650 2200 5650 2000
+Wire Wire Line
+	6000 2500 6000 2700
 Wire Wire Line
 	6000 3450 1900 3450
 Wire Wire Line
-	6000 2150 6000 1700
+	6000 2200 6000 1700
 Wire Wire Line
 	6000 1700 1800 1700
 Wire Wire Line
-	6200 5500 6900 5500
-Wire Wire Line
-	6900 5400 6200 5400
-Wire Wire Line
-	5700 5500 5100 5500
-Wire Wire Line
-	5700 5400 5450 5400
+	6100 5500 6900 5500
+Wire Wire Line
+	6900 5400 6100 5400
+Wire Wire Line
+	5800 5500 5100 5500
+Wire Wire Line
+	5800 5400 5450 5400
 Wire Wire Line
 	5450 5400 5450 5150
@@
 	8800 3250 9400 3250
 Wire Wire Line
-	8800 3350 9400 3350
+	8800 3350 9050 3350
 Wire Wire Line
 	8800 3450 9400 3450
@@
 Connection ~ 9050 3350
 Wire Wire Line
-	9050 3350 9050 2700
-$Comp
-L R R11
+	9050 3350 9050 2850
+$Comp
+L Device:R R11
 U 1 1 51E2AC95
-P 9050 2450
-F 0 "R11" H 9200 2350 40  0000 C CNN
-F 1 "10K" V 9057 2451 40  0000 C CNN
-F 2 "" V 8980 2450 30  0000 C CNN
-F 3 "" H 9050 2450 30  0000 C CNN
-	1    9050 2450
-	-1   0    0    1
-$EndComp
-Wire Wire Line
-	9050 2050 9050 2200
-$Comp
-L C C22
+P 9050 2700
+F 0 "R11" H 9200 2600 40  0000 C CNN
+F 1 "10K" V 9057 2701 40  0000 C CNN
+F 2 "" V 8980 2700 30  0000 C CNN
+F 3 "" H 9050 2700 30  0000 C CNN
+	1    9050 2700
+	-1   0    0    1
+$EndComp
+Wire Wire Line
+	9050 2200 9050 2550
+$Comp
+L Device:C C22
 U 1 1 51E2AD68
 P 6800 1750
@@
 $EndComp
 $Comp
-L C C23
+L Device:C C23
 U 1 1 51E2AD6E
 P 7200 1750
@@
 $EndComp
 Wire Wire Line
-	6800 1350 6800 1550
-Wire Wire Line
-	6800 1950 6800 2150
-Wire Wire Line
-	7200 1950 7200 2050
+	6800 1350 6800 1450
+Wire Wire Line
+	6800 1900 6800 2050
+Wire Wire Line
+	7200 1900 7200 2050
 Wire Wire Line
 	7200 2050 6800 2050
 Connection ~ 6800 2050
 Wire Wire Line
-	7200 1550 7200 1450
+	7200 1600 7200 1450
 Wire Wire Line
 	7200 1450 6800 1450
 Connection ~ 6800 1450
 $Comp
-L VSS #PWR03
+L power:VSS #PWR03
 U 1 1 51E2AE91
 P 6800 2150
 F 0 "#PWR03" H 6800 2150 30  0001 C CNN
-F 1 "VSS" H 6800 2080 30  0000 C CNN
+F 1 "VSS" H 6800 2300 30  0000 C CNN
 F 2 "" H 6800 2150 60  0000 C CNN
 F 3 "" H 6800 2150 60  0000 C CNN
 	1    6800 2150
-	1    0    0    -1
-$EndComp
-$Comp
-L C C20
+	-1   0    0    1
+$EndComp
+$Comp
+L Device:C C20
 U 1 1 51E2AF1D
 P 8250 2150
@@
 $EndComp
 $Comp
-L VSS #PWR04
+L power:VSS #PWR04
 U 1 1 51E2AF23
 P 8250 2400
 F 0 "#PWR04" H 8250 2400 30  0001 C CNN
-F 1 "VSS" H 8250 2330 30  0000 C CNN
+F 1 "VSS" H 8250 2550 30  0000 C CNN
 F 2 "" H 8250 2400 60  0000 C CNN
 F 3 "" H 8250 2400 60  0000 C CNN
 	1    8250 2400
-	1    0    0    -1
-$EndComp
-Wire Wire Line
-	8250 1900 8250 1950
-Wire Wire Line
-	8250 2350 8250 2400
-$Comp
-L VBUS #PWR05
+	-1   0    0    1
+$EndComp
+Wire Wire Line
+	8250 1900 8250 2000
+Wire Wire Line
+	8250 2300 8250 2400
+$Comp
+L freakduino:VBUS #PWR05
 U 1 1 51E361E9
 P 5450 5150
@@
 $EndComp
 $Comp
-L VCC5 #PWR06
+L freakduino:VCC5 #PWR06
 U 1 1 51E3660E
 P 5650 2000
@@
 $EndComp
 $Comp
-L VCC5 #PWR07
+L freakduino:VCC5 #PWR07
 U 1 1 51E3661D
 P 6800 1350
@@
 $EndComp
 $Comp
-L VCC5 #PWR08
+L freakduino:VCC5 #PWR08
 U 1 1 51E3662C
-P 9050 2050
-F 0 "#PWR08" H 9050 2190 20  0001 C CNN
-F 1 "VCC5" H 9050 2160 30  0000 C CNN
-F 2 "" H 9050 2050 60  0000 C CNN
-F 3 "" H 9050 2050 60  0000 C CNN
-	1    9050 2050
-	1    0    0    -1
-$EndComp
-$Comp
-L VCC5 #PWR09
+P 9050 2200
+F 0 "#PWR08" H 9050 2340 20  0001 C CNN
+F 1 "VCC5" H 9050 2310 30  0000 C CNN
+F 2 "" H 9050 2200 60  0000 C CNN
+F 3 "" H 9050 2200 60  0000 C CNN
+	1    9050 2200
+	1    0    0    -1
+$EndComp
+$Comp
+L freakduino:VCC5 #PWR09
 U 1 1 51E3663B
 P 8250 1900
@@
 $EndComp
 $Comp
-L VCC5 #PWR010
+L freakduino:VCC5 #PWR010
 U 1 1 51E3664A
 P 7700 2350
@@
 $EndComp
 $Comp
-L ATMEGA328-QFP32 U6
+L freakduino:ATMEGA328-QFP32 U6
 U 1 1 51E379D5
 P 7800 4250
 F 0 "U6" H 7100 5750 47  0000 L BNN
 F 1 "ATMEGA328-QFP32" H 8000 2650 47  0000 L BNN
-F 2 "TQFP32" H 7800 3850 59  0000 C CNB
+F 2 "TQFP32" H 7800 3850 59  0001 C CNB
 F 3 "" H 7800 4250 60  0000 C CNN
 	1    7800 4250
@@
 $EndComp
 Wire Wire Line
-	7700 5900 7700 6250
+	7700 5900 7700 6100
 Wire Wire Line
 	7800 5900 7800 6100
 Wire Wire Line
-	7500 6100 7900 6100
+	7500 6100 7700 6100
 Connection ~ 7700 6100
 Wire Wire Line
@@
 	6900 3650 6600 3650
 Wire Wire Line
-	7700 2350 7700 2650
+	7700 2350 7700 2400
 Wire Wire Line
 	7800 2650 7800 2400
 Wire Wire Line
-	7700 2400 7900 2400
+	7700 2400 7800 2400
 Connection ~ 7700 2400
 Wire Wire Line
@@
 Connection ~ 6000 3150
 Wire Wire Line
-	5550 2700 6000 2700
+	5550 2700 5650 2700
 Connection ~ 6000 2700
 Text GLabel 9400 3150 2    39   Output ~ 0
@@
 Wire Wire Line
 	7500 5900 7500 6100
+Wire Wire Line
+	5650 2700 5650 2900
+Wire Wire Line
+	5650 2700 6000 2700
+Wire Wire Line
+	4600 2900 4600 3000
+Wire Wire Line
+	9050 3350 9400 3350
+Wire Wire Line
+	6800 2050 6800 2150
+Wire Wire Line
+	6800 1450 6800 1600
+Wire Wire Line
+	7700 6100 7700 6150
+Wire Wire Line
+	7700 6100 7800 6100
+Wire Wire Line
+	7800 6100 7900 6100
+Wire Wire Line
+	7700 2400 7700 2650
+Wire Wire Line
+	7800 2400 7900 2400
+Wire Wire Line
+	6000 3150 6000 3450
+Wire Wire Line
+	6000 2700 6000 3150
 $EndSCHEMATC

Commit message: Attempting to update sch->brd netlist component footprint a for KiCAD v5+
Parts:
- C13, C20, C23: footprint (none) -> Capacitor_SMD:C_0603_1608Metric
- C22: footprint (none) -> Capacitor_SMD:C_0805_2012Metric
- R11, R13, R14, R15: footprint (none) -> Resistor_SMD:R_0603_1608Metric
- U6: footprint TQFP32 -> (none)
Changed lines of the file:
@@
 F 0 "R13" H 5800 2250 40  0000 C CNN
 F 1 "10K" V 5657 2351 40  0000 C CNN
-F 2 "" V 5580 2350 30  0000 C CNN
+F 2 "Resistor_SMD:R_0603_1608Metric" V 5580 2350 30  0001 C CNN
 F 3 "" H 5650 2350 30  0000 C CNN
 	1    5650 2350
@@
 F 0 "S2" H 5050 3200 60  0000 C CNN
 F 1 "PBS_SMD" H 5150 2550 60  0001 C CNN
-F 2 "" H 5150 2800 60  0000 C CNN
+F 2 "" H 5150 2800 60  0001 C CNN
 F 3 "" H 5150 2800 60  0000 C CNN
 	1    5150 2800
@@
 F 0 "C13" H 6000 2450 40  0000 L CNN
 F 1 "0u1" H 6006 2265 40  0000 L CNN
-F 2 "" H 6038 2200 30  0000 C CNN
+F 2 "Capacitor_SMD:C_0603_1608Metric" H 6038 2200 30  0001 C CNN
 F 3 "" H 6000 2350 60  0000 C CNN
 	1    6000 2350
@@
 Text GLabel 1900 3450 0    39   Output ~ 0
 RESET_N
-Text GLabel 1800 1700 0    39   Input ~ 0
+Text GLabel 1850 1700 0    39   Input ~ 0
 DTR_N
 Text Label 1950 1700 0    60   ~ 0
@@
 F 0 "R14" V 6030 5400 40  0000 C CNN
 F 1 "100K" V 5957 5401 40  0000 C CNN
-F 2 "" V 5880 5400 30  0000 C CNN
+F 2 "Resistor_SMD:R_0603_1608Metric" V 5880 5400 30  0001 C CNN
 F 3 "" H 5950 5400 30  0000 C CNN
 	1    5950 5400
@@
 F 0 "R15" V 5850 5500 40  0000 C CNN
 F 1 "100K" V 5957 5501 40  0000 C CNN
-F 2 "" V 5880 5500 30  0000 C CNN
+F 2 "Resistor_SMD:R_0603_1608Metric" V 5880 5500 30  0001 C CNN
 F 3 "" H 5950 5500 30  0000 C CNN
 	1    5950 5500
@@
 	6000 2200 6000 1700
 Wire Wire Line
-	6000 1700 1800 1700
+	6000 1700 1850 1700
 Wire Wire Line
 	6100 5500 6900 5500
@@
 F 0 "R11" H 9200 2600 40  0000 C CNN
 F 1 "10K" V 9057 2701 40  0000 C CNN
-F 2 "" V 8980 2700 30  0000 C CNN
+F 2 "Resistor_SMD:R_0603_1608Metric" V 8980 2700 30  0001 C CNN
 F 3 "" H 9050 2700 30  0000 C CNN
 	1    9050 2700
@@
 F 0 "C22" H 6800 1850 40  0000 L CNN
 F 1 "22u/6v3" H 6806 1665 40  0000 L CNN
-F 2 "" H 6838 1600 30  0000 C CNN
+F 2 "Capacitor_SMD:C_0805_2012Metric" H 6838 1600 30  0001 C CNN
 F 3 "" H 6800 1750 60  0000 C CNN
 	1    6800 1750
@@
 F 0 "C23" H 7200 1850 40  0000 L CNN
 F 1 "0u1" H 7206 1665 40  0000 L CNN
-F 2 "" H 7238 1600 30  0000 C CNN
+F 2 "Capacitor_SMD:C_0603_1608Metric" H 7238 1600 30  0001 C CNN
 F 3 "" H 7200 1750 60  0000 C CNN
 	1    7200 1750
@@
 F 0 "C20" H 8250 2250 40  0000 L CNN
 F 1 "0u1" H 8256 2065 40  0000 L CNN
-F 2 "" H 8288 2000 30  0000 C CNN
+F 2 "Capacitor_SMD:C_0603_1608Metric" H 8288 2000 30  0001 C CNN
 F 3 "" H 8250 2150 60  0000 C CNN
 	1    8250 2150
@@
 F 0 "U6" H 7100 5750 47  0000 L BNN
 F 1 "ATMEGA328-QFP32" H 8000 2650 47  0000 L BNN
-F 2 "TQFP32" H 7800 3850 59  0001 C CNB
+F 2 "" H 7800 3850 59  0001 C CNB
 F 3 "" H 7800 4250 60  0000 C CNN
 	1    7800 4250
