File: hardware/interface-alt.sch (KiCad schematic (older format))
At the start: 19 parts, among them SW1 DIPSW4_DIP, U4 GTL2003

Commit message: Laboriously re-worked schematic and 3D settings for KiCAD v5+
Parts:
- C18, C21: symbol C -> Device:C
- D1, D2, D6: symbol LED -> Device:LED
- H3: symbol CONN_3X2 -> Connector_Generic:Conn_02x03_Odd_Even
- JP2: symbol 1X2 -> freakduino:1X2
- JP3, JP5: symbol JP6/THRU -> Connector:Conn_01x06_Female
- JP4, JP6: symbol JP8/THRU -> Connector:Conn_01x08_Female
- R1, R10, R12, R2, R4, R5: symbol R -> Device:R
- SW1: symbol DIPSW4_DIP -> freakduino:DIPSW4_DIP
- U4: symbol GTL2003 -> freakduino:GTL2003
Connections:
- wire segments 86 -> 98

Commit message: Attempting to update sch->brd netlist component footprint a for KiCAD v5+
Parts:
- C18, C21: footprint (none) -> Capacitor_SMD:C_0603_1608Metric
- D1, D2, D6: footprint (none) -> LED_SMD:LED_0603_1608Metric
- H3: footprint (none) -> Connector_PinHeader_2.54mm:PinHeader_2x03_P2.54mm_Vertical_SMD
- JP2: footprint (none) -> Connector_PinHeader_2.54mm:PinHeader_1x02_P2.54mm_Vertical
- JP3, JP5: footprint (none) -> Connector_PinSocket_2.54mm:PinSocket_1x06_P2.54mm_Vertical
- JP4, JP6: footprint (none) -> Connector_PinSocket_2.54mm:PinSocket_1x08_P2.54mm_Vertical
- R1, R10, R12, R2, R4, R5: footprint (none) -> Resistor_SMD:R_0603_1608Metric
Changed lines of the file:
@@
 F 0 "R10" H 4550 1700 40  0000 C CNN
 F 1 "180K" V 4407 1801 40  0000 C CNN
-F 2 "" V 4330 1800 30  0000 C CNN
+F 2 "Resistor_SMD:R_0603_1608Metric" V 4330 1800 30  0001 C CNN
 F 3 "" H 4400 1800 30  0000 C CNN
 	1    4400 1800
@@
 F 0 "C21" H 3950 3800 40  0000 L CNN
 F 1 "0u1" H 3956 3615 40  0000 L CNN
-F 2 "" H 3988 3550 30  0000 C CNN
+F 2 "Capacitor_SMD:C_0603_1608Metric" H 3988 3550 30  0001 C CNN
 F 3 "" H 3950 3700 60  0000 C CNN
 	1    3950 3700
@@
 F 0 "C18" H 2550 1850 40  0000 L CNN
 F 1 "0u1" H 2556 1665 40  0000 L CNN
-F 2 "" H 2588 1600 30  0000 C CNN
+F 2 "Capacitor_SMD:C_0603_1608Metric" H 2588 1600 30  0001 C CNN
 F 3 "" H 2550 1750 60  0000 C CNN
 	1    2550 1750
@@
 $EndComp
 $Comp
-L power:VSS #PWR051
+L power:VSS #PWR0104
 U 1 1 51E3DC0E
 P 2550 2100
-F 0 "#PWR051" H 2550 2100 30  0001 C CNN
+F 0 "#PWR0104" H 2550 2100 30  0001 C CNN
 F 1 "VSS" H 2450 2100 30  0000 C CNN
 F 2 "" H 2550 2100 60  0000 C CNN
@@
 F 0 "JP2" H 4600 3750 60  0000 C CNN
 F 1 "1X2" H 4600 3650 40  0000 C CNN
-F 2 "" H 4400 3700 60  0000 C CNN
+F 2 "Connector_PinHeader_2.54mm:PinHeader_1x02_P2.54mm_Vertical" H 4400 3700 60  0001 C CNN
 F 3 "" H 4400 3700 60  0000 C CNN
 	1    4400 3700
@@
 F 0 "SW1" H 7050 3300 60  0000 L CNN
 F 1 "DIPSW4_DIP" H 7050 3100 60  0001 L CNN
-F 2 "" H 6850 3200 60  0000 C CNN
+F 2 "" H 6850 3200 60  0001 C CNN
 F 3 "" H 6850 3200 60  0000 C CNN
 	1    6850 3200
@@
 F 0 "D1" H 6450 4300 50  0000 C CNN
 F 1 "BLUE" H 6450 4100 50  0000 C CNN
-F 2 "" H 6450 4200 60  0000 C CNN
+F 2 "LED_SMD:LED_0603_1608Metric" H 6450 4200 60  0001 C CNN
 F 3 "" H 6450 4200 60  0000 C CNN
 	1    6450 4200
@@
 F 0 "D2" H 6950 4300 50  0000 C CNN
 F 1 "RED" H 6950 4100 50  0000 C CNN
-F 2 "" H 6950 4200 60  0000 C CNN
+F 2 "LED_SMD:LED_0603_1608Metric" H 6950 4200 60  0001 C CNN
 F 3 "" H 6950 4200 60  0000 C CNN
 	1    6950 4200
@@
 F 0 "R1" H 6600 5200 40  0000 C CNN
 F 1 "1K" V 6457 5301 40  0000 C CNN
-F 2 "" V 6380 5300 30  0000 C CNN
+F 2 "Resistor_SMD:R_0603_1608Metric" V 6380 5300 30  0001 C CNN
 F 3 "" H 6450 5300 30  0000 C CNN
 	1    6450 5300
@@
 F 0 "R2" H 7100 5200 40  0000 C CNN
 F 1 "1K" V 6957 5301 40  0000 C CNN
-F 2 "" V 6880 5300 30  0000 C CNN
+F 2 "Resistor_SMD:R_0603_1608Metric" V 6880 5300 30  0001 C CNN
 F 3 "" H 6950 5300 30  0000 C CNN
 	1    6950 5300
@@
 F 0 "H3" H 3600 6000 50  0000 C CNN
 F 1 "H3X2" H 3600 5950 40  0001 C CNN
-F 2 "" H 3550 6200 60  0000 C CNN
+F 2 "Connector_PinHeader_2.54mm:PinHeader_2x03_P2.54mm_Vertical_SMD" H 3550 6200 60  0001 C CNN
 F 3 "" H 3550 6200 60  0000 C CNN
 	1    3550 6200
@@
 F 0 "D6" H 7900 5050 50  0000 C CNN
 F 1 "RED" H 7900 4850 50  0000 C CNN
-F 2 "" H 7900 4950 60  0000 C CNN
+F 2 "LED_SMD:LED_0603_1608Metric" H 7900 4950 60  0001 C CNN
 F 3 "" H 7900 4950 60  0000 C CNN
 	1    7900 4950
@@
 F 0 "R12" H 8050 5400 40  0000 C CNN
 F 1 "1K" V 7907 5501 40  0000 C CNN
-F 2 "" V 7830 5500 30  0000 C CNN
+F 2 "Resistor_SMD:R_0603_1608Metric" V 7830 5500 30  0001 C CNN
 F 3 "" H 7900 5500 30  0000 C CNN
 	1    7900 5500
@@
 F 0 "R4" V 10300 2900 40  0000 C CNN
 F 1 "1K" V 10207 2901 40  0000 C CNN
-F 2 "" V 10130 2900 30  0000 C CNN
+F 2 "Resistor_SMD:R_0603_1608Metric" V 10130 2900 30  0001 C CNN
 F 3 "" H 10200 2900 30  0000 C CNN
 	1    10200 2900
@@
 F 0 "R5" V 10300 3100 40  0000 C CNN
 F 1 "1K" V 10207 3101 40  0000 C CNN
-F 2 "" V 10130 3100 30  0000 C CNN
+F 2 "Resistor_SMD:R_0603_1608Metric" V 10130 3100 30  0001 C CNN
 F 3 "" H 10200 3100 30  0000 C CNN
 	1    10200 3100
@@
 F 0 "JP3" H 10150 2000 60  0000 C CNN
 F 1 "JP6/THRU" H 10100 2350 60  0001 C CNN
-F 2 "" H 9950 2000 60  0000 C CNN
+F 2 "Connector_PinSocket_2.54mm:PinSocket_1x06_P2.54mm_Vertical" H 9950 2000 60  0001 C CNN
 F 3 "" H 9950 2000 60  0000 C CNN
 	1    9950 2000
@@
 F 0 "JP6" H 10200 3600 60  0000 C CNN
 F 1 "JP8/THRU" H 10100 4050 60  0001 C CNN
-F 2 "" H 9950 3600 60  0000 C CNN
+F 2 "Connector_PinSocket_2.54mm:PinSocket_1x08_P2.54mm_Vertical" H 9950 3600 60  0001 C CNN
 F 3 "" H 9950 3600 60  0000 C CNN
 	1    9950 3600
@@
 F 0 "JP4" H 10150 4800 60  0000 C CNN
 F 1 "JP8/THRU" H 10100 5250 60  0001 C CNN
-F 2 "" H 9950 4800 60  0000 C CNN
+F 2 "Connector_PinSocket_2.54mm:PinSocket_1x08_P2.54mm_Vertical" H 9950 4800 60  0001 C CNN
 F 3 "" H 9950 4800 60  0000 C CNN
 	1    9950 4800
@@
 F 0 "JP5" H 10100 5900 60  0000 C CNN
 F 1 "JP6/THRU" H 10100 6250 60  0001 C CNN
-F 2 "" H 9950 5900 60  0000 C CNN
+F 2 "Connector_PinSocket_2.54mm:PinSocket_1x06_P2.54mm_Vertical" H 9950 5900 60  0001 C CNN
 F 3 "" H 9950 5900 60  0000 C CNN
 	1    9950 5900
@@
 F 0 "U4" H 2800 4000 60  0000 C CNN
 F 1 "GTL2003" H 2950 2350 60  0000 C CNN
-F 2 "" H 3150 3150 60  0000 C CNN
+F 2 "" H 3150 3150 60  0001 C CNN
 F 3 "" H 3150 3150 60  0000 C CNN
 	1    3150 3150
