File: hardware/misc.sch (KiCad schematic (older format))
At the start: 5 parts

Commit message: Laboriously re-worked schematic and 3D settings for KiCAD v5+
Parts:
- H1, H2, H4, H5: symbol MOUNT_HOLE -> freakduino:MOUNT_HOLE
- JP7: symbol 1X2 -> freakduino:1X2
Connections:
- wire segments 4 -> 2
Changed lines of the file:
@@
-EESchema Schematic File Version 2
-LIBS:freakduino
-LIBS:power
-LIBS:device
-LIBS:transistors
-LIBS:conn
-LIBS:linear
-LIBS:regul
-LIBS:74xx
-LIBS:cmos4000
-LIBS:adc-dac
-LIBS:memory
-LIBS:xilinx
-LIBS:special
-LIBS:microcontrollers
-LIBS:dsp
-LIBS:microchip
-LIBS:analog_switches
-LIBS:motorola
-LIBS:texas
-LIBS:intel
-LIBS:audio
-LIBS:interface
-LIBS:digital-audio
-LIBS:philips
-LIBS:display
-LIBS:cypress
-LIBS:siliconi
-LIBS:opto
-LIBS:atmel
-LIBS:contrib
-LIBS:valves
+EESchema Schematic File Version 4
 LIBS:freakduino-alt-cache
-EELAYER 27 0
+EELAYER 26 0
 EELAYER END
 $Descr A4 11693 8268
 encoding utf-8
-Sheet 6 6
+Sheet 5 6
 Title "FREAKDUINO-CHIBI 2.4GHz"
 Date "3 mar 2014"
@@
 $EndDescr
 $Comp
-L MOUNT_HOLE H2
+L freakduino:MOUNT_HOLE H2
 U 1 1 51E3F1C3
 P 2100 1750
 F 0 "H2" H 1850 2100 60  0000 C CNN
-F 1 "MOUNT_HOLE" H 2450 1400 60  0000 C CNN
+F 1 "MOUNT_HOLE" H 2100 1300 60  0000 C CNN
 F 2 "" H 2100 1750 60  0000 C CNN
 F 3 "" H 2100 1750 60  0000 C CNN
@@
 $EndComp
 $Comp
-L MOUNT_HOLE H1
+L freakduino:MOUNT_HOLE H1
 U 1 1 51E3F2C5
 P 3700 1750
 F 0 "H1" H 3450 2100 60  0000 C CNN
-F 1 "MOUNT_HOLE" H 4050 1400 60  0000 C CNN
+F 1 "MOUNT_HOLE" H 3700 1300 60  0000 C CNN
 F 2 "" H 3700 1750 60  0000 C CNN
 F 3 "" H 3700 1750 60  0000 C CNN
@@
 $EndComp
 $Comp
-L MOUNT_HOLE H4
+L freakduino:MOUNT_HOLE H4
 U 1 1 51E3F2CB
 P 2100 3000
 F 0 "H4" H 1850 3350 60  0000 C CNN
-F 1 "MOUNT_HOLE" H 2450 2650 60  0000 C CNN
+F 1 "MOUNT_HOLE" H 2100 2550 60  0000 C CNN
 F 2 "" H 2100 3000 60  0000 C CNN
 F 3 "" H 2100 3000 60  0000 C CNN
@@
 $EndComp
 $Comp
-L MOUNT_HOLE H5
+L freakduino:MOUNT_HOLE H5
 U 1 1 51E3F2D1
 P 3700 3000
 F 0 "H5" H 3450 3350 60  0000 C CNN
-F 1 "MOUNT_HOLE" H 4050 2650 60  0000 C CNN
+F 1 "MOUNT_HOLE" H 3700 2550 60  0000 C CNN
 F 2 "" H 3700 3000 60  0000 C CNN
 F 3 "" H 3700 3000 60  0000 C CNN
@@
 NoConn ~ 2600 3000
 $Comp
-L 1X2 JP7
+L freakduino:1X2 JP7
 U 1 1 51E3F2ED
 P 3900 4500
-F 0 "JP7" H 3700 4550 60  0000 C CNN
-F 1 "1X2" H 3700 4450 40  0000 C CNN
+F 0 "JP7" V 4050 4500 60  0000 C CNN
+F 1 "1X2" V 3750 4500 40  0000 C CNN
 F 2 "" H 3900 4500 60  0000 C CNN
 F 3 "" H 3900 4500 60  0000 C CNN
 	1    3900 4500
-	1    0    0    -1
+	0    1    1    0
+$EndComp
+$Comp
+L power:VSS #PWR051
+U 1 1 51E3F303
+P 3650 4600
+F 0 "#PWR051" H 3650 4600 30  0001 C CNN
+F 1 "VSS" H 3650 4750 30  0000 C CNN
+F 2 "" H 3650 4600 60  0000 C CNN
+F 3 "" H 3650 4600 60  0000 C CNN
+	1    3650 4600
+	1    0    0    1
+$EndComp
+Text Notes 2300 4550 0    47   ~ 0
+GND TESTPOINTS FOR DEBUGGING
+Wire Wire Line
+	3650 4500 3650 4600
+$Comp
+L power:VSS #PWR?
+U 1 1 5BA2FCC7
+P 4150 4600
+F 0 "#PWR?" H 4150 4600 30  0001 C CNN
+F 1 "VSS" H 4150 4750 30  0000 C CNN
+F 2 "" H 4150 4600 60  0000 C CNN
+F 3 "" H 4150 4600 60  0000 C CNN
+	1    4150 4600
+	1    0    0    1
 $EndComp
 Wire Wire Line
-	3900 4750 3900 4950
-$Comp
-L VSS #PWR051
-U 1 1 51E3F303
-P 3900 4950
-F 0 "#PWR051" H 3900 4950 30  0001 C CNN
-F 1 "VSS" H 3900 4880 30  0000 C CNN
-F 2 "" H 3900 4950 60  0000 C CNN
-F 3 "" H 3900 4950 60  0000 C CNN
-	1    3900 4950
-	1    0    0    -1
-$EndComp
-Wire Wire Line
-	3900 4250 4100 4250
-Wire Wire Line
-	4100 4250 4100 4850
-Wire Wire Line
-	4100 4850 3900 4850
-Connection ~ 3900 4850
-Text Notes 2300 4550 0    47   ~ 0
-GND TESTPOINTS FOR DEBUGGING
+	4150 4500 4150 4600
 $EndSCHEMATC

Commit message: Attempting to update sch->brd netlist component footprint a for KiCAD v5+
Parts:
- H1, H2, H4, H5: footprint (none) -> MountingHole:MountingHole_3.2mm_M3_Pad_Via
- JP7: footprint (none) -> Connector_PinHeader_2.54mm:PinHeader_1x02_P2.54mm_Vertical
Changed lines of the file:
@@
 F 0 "H2" H 1850 2100 60  0000 C CNN
 F 1 "MOUNT_HOLE" H 2100 1300 60  0000 C CNN
-F 2 "" H 2100 1750 60  0000 C CNN
+F 2 "MountingHole:MountingHole_3.2mm_M3_Pad_Via" H 2100 1750 60  0001 C CNN
 F 3 "" H 2100 1750 60  0000 C CNN
 	1    2100 1750
@@
 F 0 "H1" H 3450 2100 60  0000 C CNN
 F 1 "MOUNT_HOLE" H 3700 1300 60  0000 C CNN
-F 2 "" H 3700 1750 60  0000 C CNN
+F 2 "MountingHole:MountingHole_3.2mm_M3_Pad_Via" H 3700 1750 60  0001 C CNN
 F 3 "" H 3700 1750 60  0000 C CNN
 	1    3700 1750
@@
 F 0 "H4" H 1850 3350 60  0000 C CNN
 F 1 "MOUNT_HOLE" H 2100 2550 60  0000 C CNN
-F 2 "" H 2100 3000 60  0000 C CNN
+F 2 "MountingHole:MountingHole_3.2mm_M3_Pad_Via" H 2100 3000 60  0001 C CNN
 F 3 "" H 2100 3000 60  0000 C CNN
 	1    2100 3000
@@
 F 0 "H5" H 3450 3350 60  0000 C CNN
 F 1 "MOUNT_HOLE" H 3700 2550 60  0000 C CNN
-F 2 "" H 3700 3000 60  0000 C CNN
+F 2 "MountingHole:MountingHole_3.2mm_M3_Pad_Via" H 3700 3000 60  0001 C CNN
 F 3 "" H 3700 3000 60  0000 C CNN
 	1    3700 3000
@@
 F 0 "JP7" V 4050 4500 60  0000 C CNN
 F 1 "1X2" V 3750 4500 40  0000 C CNN
-F 2 "" H 3900 4500 60  0000 C CNN
+F 2 "Connector_PinHeader_2.54mm:PinHeader_1x02_P2.54mm_Vertical" H 3900 4500 60  0001 C CNN
 F 3 "" H 3900 4500 60  0000 C CNN
 	1    3900 4500
@@
 	3650 4500 3650 4600
 $Comp
-L power:VSS #PWR?
+L power:VSS #PWR0103
 U 1 1 5BA2FCC7
 P 4150 4600
-F 0 "#PWR?" H 4150 4600 30  0001 C CNN
+F 0 "#PWR0103" H 4150 4600 30  0001 C CNN
 F 1 "VSS" H 4150 4750 30  0000 C CNN
 F 2 "" H 4150 4600 60  0000 C CNN
