File: hardware/power-alt.sch (KiCad schematic (older format))
At the start: 13 parts, among them J2 POWERJACK/THRU-3, U2 TC1264, U5 TPS61222

Commit message: Laboriously re-worked schematic and 3D settings for KiCAD v5+
Parts:
- BATT1, BATT2: symbol BH321-1P -> freakduino:BH321-1P
- C15, C3, C9: symbol CAPAPOL -> Device:CP
- C5: symbol C -> Device:C
- J2: symbol POWERJACK/THRU-3 -> freakduino:POWERJACK_THRU-3
- JP1: symbol JP3/THRU_VERT -> freakduino:JP3_THRU_VERT
- L2: symbol INDUCTOR_SMALL -> Device:L
- S1: symbol SW_SLIDE/THRU-3 -> freakduino:SW_SLIDE_THRU-3
- U2: symbol TC1264 -> freakduino:TC1264
- U5: symbol TPS61222 -> freakduino:TPS61222
- VR1: symbol UA78M05CDCYG3 -> freakduino:UA78M05CDCYG3
Connections:
- wire segments 45 -> 62

Commit message: Attempting to update sch->brd netlist component footprint a for KiCAD v5+
Parts:
- C15: footprint (none) -> Capacitor_SMD:C_0603_1608Metric
- C3: footprint (none) -> Capacitor_SMD:CP_Elec_5x5.8
- C5, C9: footprint (none) -> Capacitor_Tantalum_SMD:CP_EIA-2012-12_Kemet-R
- JP1: footprint (none) -> Connector_PinHeader_2.54mm:PinHeader_1x03_P2.54mm_Vertical
- L2: footprint (none) -> Inductor_SMD:L_Taiyo-Yuden_NR-40xx
Changed lines of the file:
@@
 $EndDescr
 $Comp
-L power:VSS #PWR039
+L power:VSS #PWR0101
 U 1 1 51E2B911
 P 3800 3250
-F 0 "#PWR039" H 3800 3250 30  0001 C CNN
+F 0 "#PWR0101" H 3800 3250 30  0001 C CNN
 F 1 "VSS" H 3800 3400 30  0000 C CNN
 F 2 "" H 3800 3250 60  0000 C CNN
@@
 $EndComp
 $Comp
-L power:VSS #PWR040
+L power:VSS #PWR0102
 U 1 1 51E2B959
 P 2850 3250
-F 0 "#PWR040" H 2850 3250 30  0001 C CNN
+F 0 "#PWR0102" H 2850 3250 30  0001 C CNN
 F 1 "VSS" H 2850 3400 30  0000 C CNN
 F 2 "" H 2850 3250 60  0000 C CNN
@@
 F 0 "C3" H 3250 3050 40  0000 L CNN
 F 1 "100u/16V" H 3250 2850 40  0000 L CNN
-F 2 "" H 3300 2800 30  0000 C CNN
+F 2 "Capacitor_SMD:CP_Elec_5x5.8" H 3300 2800 30  0001 C CNN
 F 3 "" H 3200 2950 300 0000 C CNN
 	1    3200 2950
@@
 F 0 "JP1" V 4950 1950 40  0000 L CNN
 F 1 "JP3/THRU_VERT" H 4850 1600 40  0001 L CNN
-F 2 "" H 4700 2200 60  0000 C CNN
+F 2 "Connector_PinHeader_2.54mm:PinHeader_1x03_P2.54mm_Vertical" H 4700 2200 60  0001 C CNN
 F 3 "" H 4700 2200 60  0000 C CNN
 	1    4700 2200
@@
 F 0 "J2" H 2300 3000 60  0000 C CNN
 F 1 "POWERJACK/THRU-3" H 2300 2550 60  0000 C CNN
-F 2 "" H 2300 2750 60  0000 C CNN
+F 2 "" H 2300 2750 60  0001 C CNN
 F 3 "" H 2300 2750 60  0000 C CNN
 	1    2300 2750
@@
 F 0 "U2" H 8400 2900 60  0000 C CNN
 F 1 "TC1264" H 8200 2250 60  0000 C CNN
-F 2 "" H 8600 2550 60  0000 C CNN
+F 2 "" H 8600 2550 60  0001 C CNN
 F 3 "" H 8600 2550 60  0000 C CNN
 	1    8600 2550
@@
 F 0 "C5" H 9400 2900 40  0000 L CNN
 F 1 "22u/6V3" H 9406 2715 40  0000 L CNN
-F 2 "" H 9438 2650 30  0000 C CNN
+F 2 "Capacitor_Tantalum_SMD:CP_EIA-2012-12_Kemet-R" H 9438 2650 30  0001 C CNN
 F 3 "" H 9400 2800 60  0000 C CNN
 	1    9400 2800
@@
 F 0 "S1" H 6700 1950 60  0000 C CNN
 F 1 "SW_SLIDE/THRU-3" H 6800 2900 60  0000 C CNN
-F 2 "" H 6750 2400 60  0000 C CNN
+F 2 "" H 6750 2400 60  0001 C CNN
 F 3 "" H 6750 2400 60  0000 C CNN
 	1    6750 2400
@@
 F 0 "L2" V 4150 4500 50  0000 C CNN
 F 1 "4.7uH" V 3950 4450 50  0000 C CNN
-F 2 "" H 4050 4500 60  0000 C CNN
+F 2 "Inductor_SMD:L_Taiyo-Yuden_NR-40xx" H 4050 4500 60  0001 C CNN
 F 3 "" H 4050 4500 60  0000 C CNN
 	1    4050 4500
@@
 F 0 "VR1" H 3800 3000 60  0000 C CNN
 F 1 "UA78M05CDCYG3" H 4250 2450 60  0000 C CNN
-F 2 "" H 3800 2700 60  0000 C CNN
+F 2 "" H 3800 2700 60  0001 C CNN
 F 3 "" H 3800 2700 60  0000 C CNN
 	1    3800 2700
@@
 F 0 "C15" H 3650 5100 40  0000 L CNN
 F 1 "10u/10V" H 3650 4900 40  0000 L CNN
-F 2 "" H 3700 4850 30  0000 C CNN
+F 2 "Capacitor_SMD:C_0603_1608Metric" H 3700 4850 30  0001 C CNN
 F 3 "" H 3600 5000 300 0000 C CNN
 	1    3600 5000
@@
 F 0 "C9" H 5750 4900 40  0000 L CNN
 F 1 "22u/16V/TANT" H 5750 4700 40  0000 L CNN
-F 2 "" H 5800 4650 30  0000 C CNN
+F 2 "Capacitor_Tantalum_SMD:CP_EIA-2012-12_Kemet-R" H 5800 4650 30  0001 C CNN
 F 3 "" H 5700 4800 300 0000 C CNN
 	1    5700 4800
@@
 F 0 "BATT1" H 2200 4400 50  0000 C CNN
 F 1 "BH321-1P" H 2200 4010 50  0000 C CNN
-F 2 "" H 2200 4200 60  0000 C CNN
+F 2 "" H 2200 4200 60  0001 C CNN
 F 3 "" H 2200 4200 60  0000 C CNN
 	1    2200 4200
@@
 F 0 "BATT2" H 2200 5000 50  0000 C CNN
 F 1 "BH321-1P" H 2200 4610 50  0000 C CNN
-F 2 "" H 2200 4800 60  0000 C CNN
+F 2 "" H 2200 4800 60  0001 C CNN
 F 3 "" H 2200 4800 60  0000 C CNN
 	1    2200 4800
@@
 F 0 "U5" H 4750 5150 60  0000 C CNN
 F 1 "TPS61222" H 4950 4350 60  0000 C CNN
-F 2 "" H 4950 4750 60  0000 C CNN
+F 2 "" H 4950 4750 60  0001 C CNN
 F 3 "" H 4950 4750 60  0000 C CNN
 	1    4950 4750
