File: hardware/radio-alt.sch (KiCad schematic (older format))
At the start: 19 parts, among them U3 AT86RF231, Y1 NX3225SA-16MHz-15ppm

Commit message: Laboriously re-worked schematic and 3D settings for KiCAD v5+
Parts:
- ANT1: symbol SMA -> freakduino:SMA
- BLN1: symbol BALUN_GRUVIN -> freakduino:BALUN_GRUVIN
- C10, C11, C12, C16, C17, C19, C2, C4, C6, C7, C8: symbol C -> Device:C
- FB1: symbol INDUCTOR_SMALL -> Device:Ferrite_Bead_Small
- L1: symbol INDUCTOR_SMALL -> Device:L
- R3, R9: symbol R -> Device:R
- U3: symbol AT86RF231 -> freakduino:AT86RF231
- Y1: symbol NX3225SA -> Device:Crystal_GND24
Connections:
- wire segments 80 -> 109

Commit message: Attempting to update sch->brd netlist component footprint a for KiCAD v5+
Parts:
- BLN1: footprint ~ -> (none)
- C10, C11, C12, C16, C17, C19, C8: footprint (none) -> Capacitor_SMD:C_0603_1608Metric
- C2, R3, R9: footprint (none) -> Resistor_SMD:R_0603_1608Metric
- C4, C6, C7: footprint (none) -> Capacitor_SMD:C_0402_1005Metric
- FB1: footprint (none) -> Inductor_SMD:L_0805_2012Metric
- L1: footprint (none) -> Inductor_SMD:L_0402_1005Metric
Changed lines of the file:
@@
 F 0 "U3" H 3750 5150 60  0000 C CNN
 F 1 "AT86RF231" H 4550 4200 60  0000 C CNN
-F 2 "" H 4450 4200 60  0000 C CNN
+F 2 "" H 4450 4200 60  0001 C CNN
 F 3 "" H 4450 4200 60  0000 C CNN
 	1    4450 4200
@@
 F 0 "FB1" V 3850 1250 50  0000 C CNN
 F 1 "FB/0805" V 4150 1250 50  0000 C CNN
-F 2 "" H 4000 1250 60  0000 C CNN
+F 2 "Inductor_SMD:L_0805_2012Metric" H 4000 1250 60  0001 C CNN
 F 3 "" H 4000 1250 60  0000 C CNN
 	1    4000 1250
@@
 F 0 "C11" H 4500 2850 40  0000 L CNN
 F 1 "0u1" H 4506 2665 40  0000 L CNN
-F 2 "" H 4538 2600 30  0000 C CNN
+F 2 "Capacitor_SMD:C_0603_1608Metric" H 4538 2600 30  0001 C CNN
 F 3 "" H 4500 2750 60  0000 C CNN
 	1    4500 2750
@@
 F 0 "C12" H 4850 2850 40  0000 L CNN
 F 1 "0u01" H 4856 2665 40  0000 L CNN
-F 2 "" H 4888 2600 30  0000 C CNN
+F 2 "Capacitor_SMD:C_0603_1608Metric" H 4888 2600 30  0001 C CNN
 F 3 "" H 4850 2750 60  0000 C CNN
 	1    4850 2750
@@
 F 0 "C8" H 5250 2850 40  0000 L CNN
 F 1 "0u01" H 5256 2665 40  0000 L CNN
-F 2 "" H 5288 2600 30  0000 C CNN
+F 2 "Capacitor_SMD:C_0603_1608Metric" H 5288 2600 30  0001 C CNN
 F 3 "" H 5250 2750 60  0000 C CNN
 	1    5250 2750
@@
 F 0 "Y1" H 1250 5400 60  0000 C CNN
 F 1 "NX3225SA-16MHz-15ppm" H 1450 4550 60  0000 C CNN
-F 2 "" H 1450 5200 60  0000 C CNN
+F 2 "" H 1450 5200 60  0001 C CNN
 F 3 "" H 1450 5200 60  0000 C CNN
 	1    1450 5200
@@
 F 0 "C17" H 1850 5500 40  0000 L CNN
 F 1 "12p" H 1856 5315 40  0000 L CNN
-F 2 "" H 1888 5250 30  0000 C CNN
+F 2 "Capacitor_SMD:C_0603_1608Metric" H 1888 5250 30  0001 C CNN
 F 3 "" H 1850 5400 60  0000 C CNN
 	1    1850 5400
@@
 F 0 "C19" H 1050 5500 40  0000 L CNN
 F 1 "12p" H 1056 5315 40  0000 L CNN
-F 2 "" H 1088 5250 30  0000 C CNN
+F 2 "Capacitor_SMD:C_0603_1608Metric" H 1088 5250 30  0001 C CNN
 F 3 "" H 1050 5400 60  0000 C CNN
 	1    1050 5400
@@
 F 0 "R9" V 2930 2950 40  0000 C CNN
 F 1 "DNI" V 2857 2951 40  0000 C CNN
-F 2 "" V 2780 2950 30  0000 C CNN
+F 2 "Resistor_SMD:R_0603_1608Metric" V 2780 2950 30  0001 C CNN
 F 3 "" H 2850 2950 30  0000 C CNN
 	1    2850 2950
@@
 F 0 "R3" V 3180 2950 40  0000 C CNN
 F 1 "DNI" V 3107 2951 40  0000 C CNN
-F 2 "" V 3030 2950 30  0000 C CNN
+F 2 "Resistor_SMD:R_0603_1608Metric" V 3030 2950 30  0001 C CNN
 F 3 "" H 3100 2950 30  0000 C CNN
 	1    3100 2950
@@
 F 0 "C7" V 6100 4100 40  0000 L CNN
 F 1 "5p6" V 6100 3800 40  0000 L CNN
-F 2 "" H 6188 3850 30  0000 C CNN
+F 2 "Capacitor_SMD:C_0402_1005Metric" H 6188 3850 30  0001 C CNN
 F 3 "" H 6150 4000 60  0000 C CNN
 	1    6150 4000
@@
 F 0 "C6" V 6100 4500 40  0000 L CNN
 F 1 "5p6" V 6100 4200 40  0000 L CNN
-F 2 "" H 6188 4250 30  0000 C CNN
+F 2 "Capacitor_SMD:C_0402_1005Metric" H 6188 4250 30  0001 C CNN
 F 3 "" H 6150 4400 60  0000 C CNN
 	1    6150 4400
@@
 F 0 "L1" V 9050 3800 50  0000 C CNN
 F 1 "3.3nH" V 8850 3800 50  0000 C CNN
-F 2 "" H 8950 3800 60  0000 C CNN
+F 2 "Inductor_SMD:L_0402_1005Metric" H 8950 3800 60  0001 C CNN
 F 3 "" H 8950 3800 60  0000 C CNN
 	1    8950 3800
@@
 F 0 "C4" H 8500 4300 40  0000 L CNN
 F 1 "0p4" H 8506 4115 40  0000 L CNN
-F 2 "" H 8538 4050 30  0000 C CNN
+F 2 "Capacitor_SMD:C_0402_1005Metric" H 8538 4050 30  0001 C CNN
 F 3 "" H 8500 4200 60  0000 C CNN
 	1    8500 4200
@@
 F 0 "C2" H 9400 4300 40  0000 L CNN
 F 1 "DNI" H 9406 4115 40  0000 L CNN
-F 2 "" H 9438 4050 30  0000 C CNN
+F 2 "Resistor_SMD:R_0603_1608Metric" H 9438 4050 30  0001 C CNN
 F 3 "" H 9400 4200 60  0000 C CNN
 	1    9400 4200
@@
 F 0 "ANT1" H 10150 4600 60  0000 C CNN
 F 1 "SMA" H 10500 4600 60  0000 C CNN
-F 2 "" H 10350 4050 60  0000 C CNN
+F 2 "" H 10350 4050 60  0001 C CNN
 F 3 "" H 10350 4050 60  0000 C CNN
 	1    10350 4050
@@
 F 0 "C16" H 3850 2850 40  0000 L CNN
 F 1 "0u1" H 3856 2665 40  0000 L CNN
-F 2 "" H 3888 2600 30  0000 C CNN
+F 2 "Capacitor_SMD:C_0603_1608Metric" H 3888 2600 30  0001 C CNN
 F 3 "" H 3850 2750 60  0000 C CNN
 	1    3850 2750
@@
 F 0 "BLN1" H 7700 4350 60  0000 L CNN
 F 1 "2450BL15B100E" H 7550 3650 60  0000 L CNN
-F 2 "~" H 7400 4200 60  0000 C CNN
+F 2 "" H 7400 4200 60  0000 C CNN
 F 3 "~" H 7400 4200 60  0000 C CNN
 	1    7400 4200
@@
 F 0 "C10" H 5250 1850 40  0000 L CNN
 F 1 "0u1" H 5256 1665 40  0000 L CNN
-F 2 "" H 5288 1600 30  0000 C CNN
+F 2 "Capacitor_SMD:C_0603_1608Metric" H 5288 1600 30  0001 C CNN
 F 3 "" H 5250 1750 60  0000 C CNN
 	1    5250 1750
