File: hardware/usb.sch (KiCad schematic (older format))
At the start: 9 parts, among them J1 USB-MINI-AB, U1 FT232-SSOP28

Commit message: Laboriously re-worked schematic and 3D settings for KiCAD v5+
Parts:
- C1, C14: symbol C -> Device:C
- D3, D4: symbol LED -> Device:LED
- J1: symbol USB-MINI-AB -> freakduino:USB-MINI-AB
- R6, R7, R8: symbol R -> Device:R
- U1: symbol FT232-SSOP28 -> freakduino:FT232-SSOP28
Connections:
- wire segments 42 -> 50
Changed lines of the file:
@@
-EESchema Schematic File Version 2
-LIBS:freakduino
-LIBS:power
-LIBS:device
-LIBS:transistors
-LIBS:conn
-LIBS:linear
-LIBS:regul
-LIBS:74xx
-LIBS:cmos4000
-LIBS:adc-dac
-LIBS:memory
-LIBS:xilinx
-LIBS:special
-LIBS:microcontrollers
-LIBS:dsp
-LIBS:microchip
-LIBS:analog_switches
-LIBS:motorola
-LIBS:texas
-LIBS:intel
-LIBS:audio
-LIBS:interface
-LIBS:digital-audio
-LIBS:philips
-LIBS:display
-LIBS:cypress
-LIBS:siliconi
-LIBS:opto
-LIBS:atmel
-LIBS:contrib
-LIBS:valves
+EESchema Schematic File Version 4
 LIBS:freakduino-alt-cache
-EELAYER 27 0
+EELAYER 26 0
 EELAYER END
 $Descr A4 11693 8268
@@
 $EndDescr
 $Comp
-L USB-MINI-AB J1
+L freakduino:USB-MINI-AB J1
 U 1 1 51E3C80C
 P 2800 3500
@@
 $EndComp
 $Comp
-L FT232-SSOP28 U1
+L freakduino:FT232-SSOP28 U1
 U 1 1 51E3CBA2
 P 5500 3900
 F 0 "U1" H 5050 5300 60  0000 C CNN
-F 1 "FT232-SSOP28" H 4850 2700 60  0000 C CNN
+F 1 "FT232-SSOP28" H 5400 4650 60  0000 C CNN
 F 2 "" H 5500 3900 60  0000 C CNN
 F 3 "" H 5500 3900 60  0000 C CNN
@@
 $EndComp
 $Comp
-L VSS #PWR030
+L power:VSS #PWR030
 U 1 1 51E3CBB5
-P 3150 4100
-F 0 "#PWR030" H 3150 4100 30  0001 C CNN
-F 1 "VSS" H 3150 4030 30  0000 C CNN
-F 2 "" H 3150 4100 60  0000 C CNN
-F 3 "" H 3150 4100 60  0000 C CNN
-	1    3150 4100
-	1    0    0    -1
+P 3150 4050
+F 0 "#PWR030" H 3150 4050 30  0001 C CNN
+F 1 "VSS" H 3150 4200 30  0000 C CNN
+F 2 "" H 3150 4050 60  0000 C CNN
+F 3 "" H 3150 4050 60  0000 C CNN
+	1    3150 4050
+	-1   0    0    1
 $EndComp
 Wire Wire Line
@@
 	3950 3700 4850 3700
 Wire Wire Line
-	3150 3700 3150 4100
+	3150 3700 3150 4000
 Wire Wire Line
 	3150 3700 3050 3700
@@
 	2650 4000 2650 3900
 Wire Wire Line
-	2350 4000 3150 4000
+	2350 4000 2450 4000
 Connection ~ 3150 4000
 Wire Wire Line
@@
 	3150 3300 3150 3050
 $Comp
-L VBUS #PWR031
+L freakduino:VBUS #PWR031
 U 1 1 51E3CC12
 P 3150 3050
@@
 DP
 $Comp
-L VSS #PWR032
+L power:VSS #PWR032
 U 1 1 51E3CC1F
 P 5300 5450
@@
 $EndComp
 Wire Wire Line
-	5300 5100 5300 5450
+	5300 5100 5300 5300
 Wire Wire Line
 	5400 5100 5400 5300
 Wire Wire Line
-	5300 5300 5750 5300
+	5300 5300 5400 5300
 Connection ~ 5300 5300
 Wire Wire Line
@@
 Connection ~ 5500 5300
 $Comp
-L VBUS #PWR033
+L freakduino:VBUS #PWR033
 U 1 1 51E3CC78
 P 5400 2200
@@
 $EndComp
 Wire Wire Line
-	5400 2200 5400 2500
+	5400 2200 5400 2300
 Wire Wire Line
 	5600 2500 5600 2300
@@
 Connection ~ 5400 2300
 $Comp
-L R R6
+L Device:R R6
 U 1 1 51E3CCB5
 P 4200 2200
@@
 	4850 2800 4200 2800
 Wire Wire Line
-	4200 2800 4200 2450
-Wire Wire Line
-	4200 1950 4200 1750
-$Comp
-L VBUS #PWR034
+	4200 2800 4200 2350
+Wire Wire Line
+	4200 2050 4200 1750
+$Comp
+L freakduino:VBUS #PWR034
 U 1 1 51E3CD0B
 P 4200 1750
@@
 FTDI_RST_N
 $Comp
-L C C14
+L Device:C C14
 U 1 1 51E3CD18
 P 6200 2000
@@
 $EndComp
 $Comp
-L VSS #PWR035
+L power:VSS #PWR035
 U 1 1 51E3CD2F
-P 6200 2300
-F 0 "#PWR035" H 6200 2300 30  0001 C CNN
-F 1 "VSS" H 6200 2230 30  0000 C CNN
-F 2 "" H 6200 2300 60  0000 C CNN
-F 3 "" H 6200 2300 60  0000 C CNN
-	1    6200 2300
-	1    0    0    -1
-$EndComp
-$Comp
-L VBUS #PWR036
+P 6200 2250
+F 0 "#PWR035" H 6200 2250 30  0001 C CNN
+F 1 "VSS" H 6200 2400 30  0000 C CNN
+F 2 "" H 6200 2250 60  0000 C CNN
+F 3 "" H 6200 2250 60  0000 C CNN
+	1    6200 2250
+	1    0    0    1
+$EndComp
+$Comp
+L freakduino:VBUS #PWR036
 U 1 1 51E3CD35
 P 6200 1750
@@
 $EndComp
 Wire Wire Line
-	6200 1750 6200 1800
-Wire Wire Line
-	6200 2200 6200 2300
+	6200 1750 6200 1850
+Wire Wire Line
+	6200 2150 6200 2250
 Wire Wire Line
 	6150 2800 6950 2800
@@
 NoConn ~ 6150 4100
 $Comp
-L LED D3
+L Device:LED D3
 U 1 1 51E3CE04
 P 7900 2850
-F 0 "D3" H 7900 2950 50  0000 C CNN
-F 1 "GREEN" H 7900 2750 50  0000 C CNN
+F 0 "D3" V 7750 2950 50  0000 C CNN
+F 1 "GREEN" V 8050 3000 50  0000 C CNN
 F 2 "" H 7900 2850 60  0000 C CNN
 F 3 "" H 7900 2850 60  0000 C CNN
@@
 $EndComp
 $Comp
-L LED D4
+L Device:LED D4
 U 1 1 51E3CE11
 P 8400 2850
-F 0 "D4" H 8400 2950 50  0000 C CNN
-F 1 "GREEN" H 8400 2750 50  0000 C CNN
+F 0 "D4" V 8250 2950 50  0000 C CNN
+F 1 "GREEN" V 8550 3000 50  0000 C CNN
 F 2 "" H 8400 2850 60  0000 C CNN
 F 3 "" H 8400 2850 60  0000 C CNN
@@
 $EndComp
 $Comp
-L R R7
+L Device:R R7
 U 1 1 51E3CE2B
 P 7900 3450
@@
 $EndComp
 $Comp
-L R R8
+L Device:R R8
 U 1 1 51E3CE31
 P 8400 3450
@@
 $EndComp
 Wire Wire Line
-	7900 3200 7900 3050
-Wire Wire Line
-	8400 3050 8400 3200
-Wire Wire Line
-	7900 3700 7900 3900
+	7900 3300 7900 3000
+Wire Wire Line
+	8400 3000 8400 3300
+Wire Wire Line
+	7900 3600 7900 3900
 Wire Wire Line
 	7900 3900 6150 3900
@@
 	6150 4000 8400 4000
 Wire Wire Line
-	8400 4000 8400 3700
-$Comp
-L VBUS #PWR037
+	8400 4000 8400 3600
+$Comp
+L freakduino:VBUS #PWR037
 U 1 1 51E3CEEA
 P 7900 2450
@@
 $EndComp
 $Comp
-L VBUS #PWR038
+L freakduino:VBUS #PWR038
 U 1 1 51E3CEF0
 P 8400 2450
@@
 $EndComp
 Wire Wire Line
-	7900 2650 7900 2450
-Wire Wire Line
-	8400 2450 8400 2650
+	7900 2700 7900 2450
+Wire Wire Line
+	8400 2450 8400 2700
 NoConn ~ 4850 4600
 NoConn ~ 4850 4500
@@
 RXLED_N
 $Comp
-L C C1
+L Device:C C1
 U 1 1 51E3D2B0
 P 4150 4400
@@
 USB_3V3OUT
 $Comp
-L VSS #PWR039
+L power:VSS #PWR039
 U 1 1 51E3D7CC
-P 6450 4650
-F 0 "#PWR039" H 6450 4650 30  0001 C CNN
-F 1 "VSS" H 6450 4580 30  0000 C CNN
-F 2 "" H 6450 4650 60  0000 C CNN
-F 3 "" H 6450 4650 60  0000 C CNN
-	1    6450 4650
-	1    0    0    -1
-$EndComp
-Wire Wire Line
-	6450 4650 6450 4500
+P 6450 4550
+F 0 "#PWR039" H 6450 4550 30  0001 C CNN
+F 1 "VSS" H 6450 4700 30  0000 C CNN
+F 2 "" H 6450 4550 60  0000 C CNN
+F 3 "" H 6450 4550 60  0000 C CNN
+	1    6450 4550
+	1    0    0    1
+$EndComp
+Wire Wire Line
+	6450 4550 6450 4500
 Wire Wire Line
 	6450 4500 6150 4500
@@
 NoConn ~ 6150 4600
 Wire Wire Line
-	4150 4750 4150 4600
+	4150 4700 4150 4550
 Wire Wire Line
 	4850 4100 4150 4100
 Wire Wire Line
-	4150 4100 4150 4200
-$Comp
-L VSS #PWR040
+	4150 4100 4150 4250
+$Comp
+L power:VSS #PWR040
 U 1 1 51E3D2B6
-P 4150 4750
-F 0 "#PWR040" H 4150 4750 30  0001 C CNN
-F 1 "VSS" H 4150 4680 30  0000 C CNN
-F 2 "" H 4150 4750 60  0000 C CNN
-F 3 "" H 4150 4750 60  0000 C CNN
-	1    4150 4750
-	1    0    0    -1
-$EndComp
+P 4150 4700
+F 0 "#PWR040" H 4150 4700 30  0001 C CNN
+F 1 "VSS" H 4150 4850 30  0000 C CNN
+F 2 "" H 4150 4700 60  0000 C CNN
+F 3 "" H 4150 4700 60  0000 C CNN
+	1    4150 4700
+	1    0    0    1
+$EndComp
+Wire Wire Line
+	3150 4000 3150 4050
+Wire Wire Line
+	2650 4000 3150 4000
+Wire Wire Line
+	2550 4000 2650 4000
+Wire Wire Line
+	2450 4000 2550 4000
+Wire Wire Line
+	5300 5300 5300 5450
+Wire Wire Line
+	5400 5300 5500 5300
+Wire Wire Line
+	5500 5300 5750 5300
+Wire Wire Line
+	5400 2300 5400 2500
 $EndSCHEMATC

Commit message: Attempting to update sch->brd netlist component footprint a for KiCAD v5+
Parts:
- C1, C14: footprint (none) -> Capacitor_SMD:C_0603_1608Metric
- D3, D4: footprint (none) -> LED_SMD:LED_0603_1608Metric
- R6, R7, R8: footprint (none) -> Resistor_SMD:R_0603_1608Metric
Changed lines of the file:
@@
 F 0 "J1" H 2900 3850 60  0000 C CNN
 F 1 "USB-MINI-AB" H 2400 3850 60  0000 C CNN
-F 2 "" H 2800 3500 60  0000 C CNN
+F 2 "" H 2800 3500 60  0001 C CNN
 F 3 "" H 2800 3500 60  0000 C CNN
 	1    2800 3500
@@
 F 0 "U1" H 5050 5300 60  0000 C CNN
 F 1 "FT232-SSOP28" H 5400 4650 60  0000 C CNN
-F 2 "" H 5500 3900 60  0000 C CNN
+F 2 "" H 5500 3900 60  0001 C CNN
 F 3 "" H 5500 3900 60  0000 C CNN
 	1    5500 3900
@@
 F 0 "R6" V 4280 2200 40  0000 C CNN
 F 1 "10K" V 4207 2201 40  0000 C CNN
-F 2 "" V 4130 2200 30  0000 C CNN
+F 2 "Resistor_SMD:R_0603_1608Metric" V 4130 2200 30  0001 C CNN
 F 3 "" H 4200 2200 30  0000 C CNN
 	1    4200 2200
@@
 F 0 "C14" H 6200 2100 40  0000 L CNN
 F 1 "0u1" H 6206 1915 40  0000 L CNN
-F 2 "" H 6238 1850 30  0000 C CNN
+F 2 "Capacitor_SMD:C_0603_1608Metric" H 6238 1850 30  0001 C CNN
 F 3 "" H 6200 2000 60  0000 C CNN
 	1    6200 2000
@@
 F 0 "D3" V 7750 2950 50  0000 C CNN
 F 1 "GREEN" V 8050 3000 50  0000 C CNN
-F 2 "" H 7900 2850 60  0000 C CNN
+F 2 "LED_SMD:LED_0603_1608Metric" H 7900 2850 60  0001 C CNN
 F 3 "" H 7900 2850 60  0000 C CNN
 	1    7900 2850
@@
 F 0 "D4" V 8250 2950 50  0000 C CNN
 F 1 "GREEN" V 8550 3000 50  0000 C CNN
-F 2 "" H 8400 2850 60  0000 C CNN
+F 2 "LED_SMD:LED_0603_1608Metric" H 8400 2850 60  0001 C CNN
 F 3 "" H 8400 2850 60  0000 C CNN
 	1    8400 2850
@@
 F 0 "R7" V 7980 3450 40  0000 C CNN
 F 1 "1K" V 7907 3451 40  0000 C CNN
-F 2 "" V 7830 3450 30  0000 C CNN
+F 2 "Resistor_SMD:R_0603_1608Metric" V 7830 3450 30  0001 C CNN
 F 3 "" H 7900 3450 30  0000 C CNN
 	1    7900 3450
@@
 F 0 "R8" V 8480 3450 40  0000 C CNN
 F 1 "1K" V 8407 3451 40  0000 C CNN
-F 2 "" V 8330 3450 30  0000 C CNN
+F 2 "Resistor_SMD:R_0603_1608Metric" V 8330 3450 30  0001 C CNN
 F 3 "" H 8400 3450 30  0000 C CNN
 	1    8400 3450
@@
 F 0 "C1" H 4150 4500 40  0000 L CNN
 F 1 "0u1" H 4156 4315 40  0000 L CNN
-F 2 "" H 4188 4250 30  0000 C CNN
+F 2 "Capacitor_SMD:C_0603_1608Metric" H 4188 4250 30  0001 C CNN
 F 3 "" H 4150 4400 60  0000 C CNN
 	1    4150 4400
